File: PCB/Hackpad.kicad_pcb (KiCad board)
At the start: 2 copper layers, 92.5 x 42 mm, 35 parts, among them SW1 SW_Push_45deg, SW2 SW_Push_45deg, SW3 SW_Push_45deg, SW4 SW_Push_45deg, SW5 SW_Push_45deg, SW7 SW_Push_45deg, SW8 SW_Push_45deg, U1 XIAO-RP2040-DIP

Commit message: added text
Other:
- board text added: "The-Wolf MIDI (Pro) Pad"
- board text added: "XIAO Here"
Changed lines of the file:
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@@
 		(layer "Edge.Cuts")
+	)
+	(gr_text "The-Wolf\nMIDI (Pro) Pad"
+		(at 180 134.5 0)
+		(layer "F.SilkS")
+		(effects
+			(font
+				(size 1 1)
+				(thickness 0.1)
+			)
+			(justify left bottom)
+		)
+	)
+	(gr_text "XIAO Here"
+		(at 181.5 102 0)
+		(layer "F.SilkS")
+		(effects
+			(font
+				(size 1 1)
+				(thickness 0.15)
+			)
+			(justify left bottom)
+		)
 	)
 	(segment
